File: dalekFoot/pcb/wheel/wheel.sch (EAGLE design)
At the start: 72 parts, among them IC1 LM1117MP-3.3, IC2 LM1117MP-3.3, IC3 LM1117MP-3.3, IC4 4051D, IC5 4051D, K1 12X12-TACTILE, K2 12X12-TACTILE, K3 12X12-TACTILE, K4 12X12-TACTILE, K5 12X12-TACTILE, U1 TB6612FNG(O,C,8,EL, U2 SS8050-SOT-23, U3 SS8050-SOT-23, U4 SS8050-SOT-23, U5 TB6612FNG(O,C,8,EL, U6 TB6612FNG(O,C,8,EL

Commit message: bugfix: to avoid conflict of STMF4 break board
Connections:
- removed net PA8: R29.P$1, U$1.P$A8
- removed net PB10: JP6.4, U$1.P$B10
- removed net PB11: JP6.6, U$1.P$B11
- new net BUZZER: R29.P$1, U$1.P$A11
- new net DIN1: JP6.3, U$1.P$E5
- new net DIN2: JP6.5, U$1.P$E6
- new net DIN3: JP6.4, U$1.P$E7
- new net DIN4: JP6.6, U$1.P$E8
- new net I2C2_SCL: JP5.3, U$1.P$B10
- new net I2C2_SDA: JP5.5, U$1.P$B11
- new net I2C3_SCL: JP5.4, U$1.P$A8
- new net I2C3_SDA: JP5.6, U$1.P$C9
- net PB4: no longer JP5.3
- net PB5: no longer JP5.5
- net PB6: no longer JP5.4
- net PB7: no longer JP5.6
- net PB8: no longer JP6.3
- net PB9: no longer JP6.5
- net PWM3.B: now also U$1.P$A15; no longer U$1.P$C9
Changed lines of the file:
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@@
 <label x="309.88" y="83.82" size="1.778" layer="95"/>
-</segment>
-<segment>
-<pinref part="JP6" gate="A" pin="3"/>
-<wire x1="312.42" y1="426.72" x2="325.12" y2="426.72" width="0.1524" layer="91"/>
-<label x="312.42" y="426.72" size="1.778" layer="95"/>
 </segment>
 </net>
@@
 <label x="309.88" y="81.28" size="1.778" layer="95"/>
 </segment>
-<segment>
-<pinref part="JP6" gate="A" pin="5"/>
-<wire x1="325.12" y1="424.18" x2="312.42" y2="424.18" width="0.1524" layer="91"/>
-<label x="312.42" y="424.18" size="1.778" layer="95"/>
-</segment>
-</net>
-<net name="PB10" class="0">
-<segment>
-<pinref part="U$1" gate="G$1" pin="P$B10"/>
-<wire x1="307.34" y1="78.74" x2="317.5" y2="78.74" width="0.1524" layer="91"/>
-<label x="309.88" y="78.74" size="1.778" layer="95"/>
-</segment>
-<segment>
-<pinref part="JP6" gate="A" pin="4"/>
-<wire x1="332.74" y1="426.72" x2="347.98" y2="426.72" width="0.1524" layer="91"/>
-<label x="342.9" y="426.72" size="1.778" layer="95"/>
-</segment>
-</net>
-<net name="PB11" class="0">
-<segment>
-<pinref part="U$1" gate="G$1" pin="P$B11"/>
-<wire x1="307.34" y1="76.2" x2="317.5" y2="76.2" width="0.1524" layer="91"/>
-<label x="309.88" y="76.2" size="1.778" layer="95"/>
-</segment>
-<segment>
-<pinref part="JP6" gate="A" pin="6"/>
-<wire x1="332.74" y1="424.18" x2="347.98" y2="424.18" width="0.1524" layer="91"/>
-<label x="342.9" y="424.18" size="1.778" layer="95"/>
-</segment>
 </net>
 <net name="PB4" class="0">
@@
 <label x="309.88" y="93.98" size="1.778" layer="95"/>
 </segment>
-<segment>
-<pinref part="JP5" gate="A" pin="3"/>
-<wire x1="284.48" y1="426.72" x2="269.24" y2="426.72" width="0.1524" layer="91"/>
-<label x="269.24" y="426.72" size="1.778" layer="95"/>
-</segment>
 </net>
 <net name="PB5" class="0">
@@
 <label x="309.88" y="91.44" size="1.778" layer="95"/>
 </segment>
-<segment>
-<pinref part="JP5" gate="A" pin="5"/>
-<wire x1="269.24" y1="424.18" x2="284.48" y2="424.18" width="0.1524" layer="91"/>
-<label x="269.24" y="424.18" size="1.778" layer="95"/>
-</segment>
 </net>
 <net name="PB6" class="0">
@@
 <label x="309.88" y="88.9" size="1.778" layer="95"/>
 </segment>
-<segment>
-<pinref part="JP5" gate="A" pin="4"/>
-<wire x1="292.1" y1="426.72" x2="307.34" y2="426.72" width="0.1524" layer="91"/>
-<label x="299.72" y="426.72" size="1.778" layer="95"/>
-</segment>
 </net>
 <net name="PB7" class="0">
@@
 <wire x1="307.34" y1="86.36" x2="317.5" y2="86.36" width="0.1524" layer="91"/>
 <label x="309.88" y="86.36" size="1.778" layer="95"/>
-</segment>
-<segment>
-<pinref part="JP5" gate="A" pin="6"/>
-<wire x1="292.1" y1="424.18" x2="307.34" y2="424.18" width="0.1524" layer="91"/>
-<label x="299.72" y="424.18" size="1.778" layer="95"/>
 </segment>
 </net>
@@
 </segment>
 </net>
-<net name="PA8" class="0">
+<net name="I2C3_SCL" class="0">
 <segment>
 <pinref part="U$1" gate="G$1" pin="P$A8"/>
@@
 </segment>
 <segment>
-<pinref part="R29" gate="G$1" pin="P$1"/>
-<wire x1="20.32" y1="431.8" x2="12.7" y2="431.8" width="0.1524" layer="91"/>
-<label x="15.24" y="431.8" size="1.778" layer="95"/>
+<pinref part="JP5" gate="A" pin="4"/>
+<wire x1="292.1" y1="426.72" x2="307.34" y2="426.72" width="0.1524" layer="91"/>
+<label x="299.72" y="426.72" size="1.778" layer="95"/>
 </segment>
 </net>
@@
 <net name="PWM3.B" class="0">
 <segment>
-<pinref part="U$1" gate="G$1" pin="P$C9"/>
-<wire x1="330.2" y1="81.28" x2="337.82" y2="81.28" width="0.1524" layer="91"/>
-<label x="332.74" y="81.28" size="1.778" layer="95"/>
-</segment>
-<segment>
 <pinref part="U6" gate="G$1" pin="PWMB"/>
 <wire x1="251.46" y1="607.06" x2="266.7" y2="607.06" width="0.1524" layer="91"/>
 <label x="251.46" y="607.06" size="1.778" layer="95"/>
+</segment>
+<segment>
+<pinref part="U$1" gate="G$1" pin="P$A15"/>
+<wire x1="281.94" y1="66.04" x2="292.1" y2="66.04" width="0.1524" layer="91"/>
+<label x="284.48" y="66.04" size="1.778" layer="95"/>
 </segment>
 </net>
@@
 </segment>
 </net>
+<net name="BUZZER" class="0">
+<segment>
+<pinref part="U$1" gate="G$1" pin="P$A11"/>
+<wire x1="281.94" y1="76.2" x2="292.1" y2="76.2" width="0.1524" layer="91"/>
+<label x="284.48" y="76.2" size="1.778" layer="95"/>
+</segment>
+<segment>
+<pinref part="R29" gate="G$1" pin="P$1"/>
+<wire x1="20.32" y1="431.8" x2="12.7" y2="431.8" width="0.1524" layer="91"/>
+<label x="15.24" y="431.8" size="1.778" layer="95"/>
+</segment>
+</net>
+<net name="I2C3_SDA" class="0">
+<segment>
+<pinref part="U$1" gate="G$1" pin="P$C9"/>
+<wire x1="330.2" y1="81.28" x2="337.82" y2="81.28" width="0.1524" layer="91"/>
+<label x="332.74" y="81.28" size="1.778" layer="95"/>
+</segment>
+<segment>
+<pinref part="JP5" gate="A" pin="6"/>
+<wire x1="292.1" y1="424.18" x2="307.34" y2="424.18" width="0.1524" layer="91"/>
+<label x="299.72" y="424.18" size="1.778" layer="95"/>
+</segment>
+</net>
+<net name="I2C2_SCL" class="0">
+<segment>
+<pinref part="U$1" gate="G$1" pin="P$B10"/>
+<wire x1="307.34" y1="78.74" x2="317.5" y2="78.74" width="0.1524" layer="91"/>
+<label x="309.88" y="78.74" size="1.778" layer="95"/>
+</segment>
+<segment>
+<pinref part="JP5" gate="A" pin="3"/>
+<wire x1="284.48" y1="426.72" x2="269.24" y2="426.72" width="0.1524" layer="91"/>
+<label x="269.24" y="426.72" size="1.778" layer="95"/>
+</segment>
+</net>
+<net name="I2C2_SDA" class="0">
+<segment>
+<pinref part="U$1" gate="G$1" pin="P$B11"/>
+<wire x1="307.34" y1="76.2" x2="317.5" y2="76.2" width="0.1524" layer="91"/>
+<label x="309.88" y="76.2" size="1.778" layer="95"/>
+</segment>
+<segment>
+<pinref part="JP5" gate="A" pin="5"/>
+<wire x1="269.24" y1="424.18" x2="284.48" y2="424.18" width="0.1524" layer="91"/>
+<label x="269.24" y="424.18" size="1.778" layer="95"/>
+</segment>
+</net>
+<net name="DIN1" class="0">
+<segment>
+<pinref part="U$1" gate="G$1" pin="P$E5"/>
+<wire x1="375.92" y1="91.44" x2="391.16" y2="91.44" width="0.1524" layer="91"/>
+<label x="378.46" y="91.44" size="1.778" layer="95"/>
+</segment>
+<segment>
+<pinref part="JP6" gate="A" pin="3"/>
+<wire x1="312.42" y1="426.72" x2="325.12" y2="426.72" width="0.1524" layer="91"/>
+<label x="312.42" y="426.72" size="1.778" layer="95"/>
+</segment>
+</net>
+<net name="DIN2" class="0">
+<segment>
+<pinref part="U$1" gate="G$1" pin="P$E6"/>
+<wire x1="375.92" y1="88.9" x2="391.16" y2="88.9" width="0.1524" layer="91"/>
+<label x="378.46" y="88.9" size="1.778" layer="95"/>
+</segment>
+<segment>
+<pinref part="JP6" gate="A" pin="5"/>
+<wire x1="325.12" y1="424.18" x2="312.42" y2="424.18" width="0.1524" layer="91"/>
+<label x="312.42" y="424.18" size="1.778" layer="95"/>
+</segment>
+</net>
+<net name="DIN3" class="0">
+<segment>
+<pinref part="U$1" gate="G$1" pin="P$E7"/>
+<wire x1="375.92" y1="86.36" x2="391.16" y2="86.36" width="0.1524" layer="91"/>
+<label x="378.46" y="86.36" size="1.778" layer="95"/>
+</segment>
+<segment>
+<pinref part="JP6" gate="A" pin="4"/>
+<wire x1="332.74" y1="426.72" x2="347.98" y2="426.72" width="0.1524" layer="91"/>
+<label x="342.9" y="426.72" size="1.778" layer="95"/>
+</segment>
+</net>
+<net name="DIN4" class="0">
+<segment>
+<pinref part="U$1" gate="G$1" pin="P$E8"/>
+<wire x1="375.92" y1="83.82" x2="391.16" y2="83.82" width="0.1524" layer="91"/>
+<label x="378.46" y="83.82" size="1.778" layer="95"/>
+</segment>
+<segment>
+<pinref part="JP6" gate="A" pin="6"/>
+<wire x1="332.74" y1="424.18" x2="347.98" y2="424.18" width="0.1524" layer="91"/>
+<label x="342.9" y="424.18" size="1.778" layer="95"/>
+</segment>
+</net>

Commit message: bugfix: fix 4051 addr pin missing
Parts:
- added C8: 10uf, rcl:CPOL-US153CLV-0505
- added C9: 100uf, rcl:CPOL-US153CLV-0605
- added D4: (no value), diode:DIODE-DO-214AC
- added IC6: LM1117MP-3.3, lm1117:LM1117MP-3.3
- added JP7: (no value), pinhead:PINHD-2X8
- added R35: (no value), hqc:R-0805
Connections:
- removed net N$25: U$1.P$C10
- removed net N$26: U$1.P$C11
- removed net N$27: U$1.P$C12
- removed net N$56: IC4A.A
- removed net N$57: IC4A.B
- removed net N$58: IC4A.C
- removed net N$59: IC5A.A
- removed net N$60: IC5A.B
- removed net N$61: IC5A.C
- removed net VCC-DIGITAL: B1.P$+, C2.+, IC1.OUT, JP5.1, JP5.2, JP6.1, JP6.2, LED1.A, LED2.A, R27.1, R28.1, U$1.P$3V3, U1.STBY, U1.VCC, U5.STBY, U5.VCC, U6.STBY, U6.VCC
- new net MADC_A: IC4A.A, IC5A.A, U$1.P$C10
- new net MADC_B: IC4A.B, IC5A.B, U$1.P$C11
- new net MADC_C: IC4A.C, IC5A.C, U$1.P$C12
- new net N$2: D4.C, IC6.IN
- new net N$6: JP7.1, JP7.11, JP7.13, JP7.15, JP7.3, JP7.5, JP7.7, JP7.9, R35.P$2
- new net VCC-IRT: B1.P$+, C2.+, C9.+, IC1.OUT, IC6.OUT, JP5.1, JP5.2, JP6.1, JP6.2, LED1.A, LED2.A, R27.1, R28.1, R35.P$1, U$1.P$3V3, U1.STBY, U1.VCC, U5.STBY, U5.VCC, U6.STBY, U6.VCC
- net BAT+: now also C8.+, D4.A
- net DGND: now also C8.-, C9.-, IC6.GND, JP7.10, JP7.12, JP7.14, JP7.16, JP7.2, JP7.4, JP7.6, JP7.8
